File: TinyGame_RC1/TinyGame RC1_Jig.sch (EAGLE design)
At the start: 42 parts, among them K1 BUTTON-4P-3100010P1, K2 BUTTON-4P-3100010P1

Commit message: Artwork and gerbers
Parts:
- added U$2: TINRS_ARTWORKLOGO, EurorackModularParts:TINRS_ARTWORKLOGO
- added U$3: TINRS_ARTWORKROCKET, EurorackModularParts:TINRS_ARTWORKROCKET
Changed lines of the file:
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@@
 <?xml version="1.0" encoding="utf-8"?>
 <!DOCTYPE eagle SYSTEM "eagle.dtd">
-<eagle version="6.5.0">
+<eagle version="7.7.0">
 <drawing>
 <settings>
@@
 <setting verticaltext="up"/>
 </settings>
-<grid distance="0.05" unitdist="inch" unit="inch" style="lines" multiple="1" display="no" altdistance="0.01" altunitdist="inch" altunit="inch"/>
+<grid distance="0.1" unitdist="inch" unit="inch" style="lines" multiple="1" display="no" altdistance="0.01" altunitdist="inch" altunit="inch"/>
 <layers>
 <layer number="1" name="Top" color="4" fill="1" visible="no" active="no"/>
@@
 <part name="R8" library="OPL" deviceset="R*" device="-0603" value="10K"/>
 <part name="SUPPLY6" library="SparkFun-Aesthetics" deviceset="3.3V" device=""/>
+<part name="U$2" library="EurorackModularParts" deviceset="TINRS_ARTWORK" device="LOGO"/>
+<part name="U$3" library="EurorackModularParts" deviceset="TINRS_ARTWORK" device="ROCKET"/>
 </parts>
 <sheets>
@@
 <instance part="R8" gate="R" x="30.48" y="85.09" rot="R270"/>
 <instance part="SUPPLY6" gate="G$1" x="35.56" y="78.74" rot="R180"/>
+<instance part="U$2" gate="G$1" x="22.86" y="167.64"/>
+<instance part="U$3" gate="G$1" x="27.94" y="152.4"/>
 </instances>
 <busses>
